Commit message: 0826 update

File: install/hr_description/share/hr_description/urdf/hr.ros2_control.xacro (robot description, xacro)
@@ -8,4 +8,5 @@
     initial_positions:=${dict(shoulder_pan_joint=0.0,shoulder_lift_joint=-1.57,elbow_joint=0.0,wrist_1_joint=-1.57,wrist_2_joint=0.0,wrist_3_joint=0.0)}
     tf_prefix
+    use_conveyor_belt:=false
     ">
     <ros2_control name="${name}" type="system">
@@ -21,4 +22,16 @@
         </xacro:if>
       </hardware>
+      <!-- Add conveyor belt joint if use_conveyor_belt is true -->
+      <xacro:if value="${use_conveyor_belt}">
+        <joint name="${tf_prefix}conveyor_to_robot_base">
+          <command_interface name="position"/>
+          <command_interface name="velocity"/>
+          <state_interface name="position">
+            <param name="initial_value">0.0</param>
+          </state_interface>
+          <state_interface name="velocity"/>
+          <state_interface name="effort"/>
+        </joint>
+      </xacro:if>
       <joint name="${tf_prefix}shoulder_pan_joint">
         <command_interface name="position"/>
@@ -81,137 +94,4 @@
         <state_interface name="effort"/>
       </joint>
-      <xacro:unless value="${sim_gazebo or sim_ignition}">
-        <sensor name="${tf_prefix}tcp_fts_sensor">
-          <state_interface name="force.x"/>
-          <state_interface name="force.y"/>
-          <state_interface name="force.z"/>
-          <state_interface name="torque.x"/>
-          <state_interface name="torque.y"/>
-          <state_interface name="torque.z"/>
-        </sensor>
-        <!-- NOTE The following are joints used only for testing with fake hardware and will change in the future -->
-        <gpio name="${tf_prefix}speed_scaling">
-          <state_interface name="speed_scaling_factor"/>
-          <param name="initial_speed_scaling_factor">1</param>
-          <command_interface name="target_speed_fraction_cmd"/>
-          <command_interface name="target_speed_fraction_async_success"/>
-        </gpio>
-        <gpio name="${tf_prefix}gpio">
-          <command_interface name="standard_digital_output_cmd_0"/>
-          <command_interface name="standard_digital_output_cmd_1"/>
-          <command_interface name="standard_digital_output_cmd_2"/>
-          <command_interface name="standard_digital_output_cmd_3"/>
-          <command_interface name="standard_digital_output_cmd_4"/>
-          <command_interface name="standard_digital_output_cmd_5"/>
-          <command_interface name="standard_digital_output_cmd_6"/>
-          <command_interface name="standard_digital_output_cmd_7"/>
-          <command_interface name="standard_digital_output_cmd_8"/>
-          <command_interface name="standard_digital_output_cmd_9"/>
-          <command_interface name="standard_digital_output_cmd_10"/>
-          <command_interface name="standard_digital_output_cmd_11"/>
-          <command_interface name="standard_digital_output_cmd_12"/>
-          <command_interface name="standard_digital_output_cmd_13"/>
-          <command_interface name="standard_digital_output_cmd_14"/>
-          <command_interface name="standard_digital_output_cmd_15"/>
-          <command_interface name="standard_digital_output_cmd_16"/>
-          <command_interface name="standard_digital_output_cmd_17"/>
-          <command_interface name="standard_analog_output_cmd_0"/>
-          <command_interface name="standard_analog_output_cmd_1"/>
-          <command_interface name="tool_voltage_cmd"/>
-          <command_interface name="io_async_success"/>
-          <state_interface name="digital_output_0"/>
-          <state_interface name="digital_output_1"/>
-          <state_interface name="digital_output_2"/>
-          <state_interface name="digital_output_3"/>
-          <state_interface name="digital_output_4"/>
-          <state_interface name="digital_output_5"/>
-          <state_interface name="digital_output_6"/>
-          <state_interface name="digital_output_7"/>
-          <state_interface name="digital_output_8"/>
-          <state_interface name="digital_output_9"/>
-          <state_interface name="digital_output_10"/>
-          <state_interface name="digital_output_11"/>
-          <state_interface name="digital_output_12"/>
-          <state_interface name="digital_output_13"/>
-          <state_interface name="digital_output_14"/>
-          <state_interface name="digital_output_15"/>
-          <state_interface name="digital_output_16"/>
-          <state_interface name="digital_output_17"/>
-          <state_interface name="digital_input_0"/>
-          <state_interface name="digital_input_1"/>
-          <state_interface name="digital_input_2"/>
-          <state_interface name="digital_input_3"/>
-          <state_interface name="digital_input_4"/>
-          <state_interface name="digital_input_5"/>
-          <state_interface name="digital_input_6"/>
-          <state_interface name="digital_input_7"/>
-          <state_interface name="digital_input_8"/>
-          <state_interface name="digital_input_9"/>
-          <state_interface name="digital_input_10"/>
-          <state_interface name="digital_input_11"/>
-          <state_interface name="digital_input_12"/>
-          <state_interface name="digital_input_13"/>
-          <state_interface name="digital_input_14"/>
-          <state_interface name="digital_input_15"/>
-          <state_interface name="digital_input_16"/>
-          <state_interface name="digital_input_17"/>
-          <state_interface name="standard_analog_output_0"/>
-          <state_interface name="standard_analog_output_1"/>
-          <state_interface name="standard_analog_input_0"/>
-          <state_interface name="standard_analog_input_1"/>
-          <state_interface name="analog_io_type_0"/>
-          <state_interface name="analog_io_type_1"/>
-          <state_interface name="analog_io_type_2"/>
-          <state_interface name="analog_io_type_3"/>
-          <state_interface name="tool_mode"/>
-          <state_interface name="tool_output_voltage"/>
-          <state_interface name="tool_output_current"/>
-          <state_interface name="tool_temperature"/>
-          <state_interface name="tool_analog_input_0"/>
-          <state_interface name="tool_analog_input_1"/>
-          <state_interface name="tool_analog_input_type_0"/>
-          <state_interface name="tool_analog_input_type_1"/>
-          <state_interface name="robot_mode"/>
-          <state_interface name="robot_status_bit_0"/>
-          <state_interface name="robot_status_bit_1"/>
-          <state_interface name="robot_status_bit_2"/>
-          <state_interface name="robot_status_bit_3"/>
-          <state_interface name="safety_mode"/>
-          <state_interface name="safety_status_bit_0"/>
-          <state_interface name="safety_status_bit_1"/>
-          <state_interface name="safety_status_bit_2"/>
-          <state_interface name="safety_status_bit_3"/>
-          <state_interface name="safety_status_bit_4"/>
-          <state_interface name="safety_status_bit_5"/>
-          <state_interface name="safety_status_bit_6"/>
-          <state_interface name="safety_status_bit_7"/>
-          <state_interface name="safety_status_bit_8"/>
-          <state_interface name="safety_status_bit_9"/>
-          <state_interface name="safety_status_bit_10"/>
-          <state_interface name="program_running"/>
-        </gpio>
-        <gpio name="${tf_prefix}payload">
-          <command_interface name="mass"/>
-          <command_interface name="cog.x"/>
-          <command_interface name="cog.y"/>
-          <command_interface name="cog.z"/>
-          <command_interface name="payload_async_success"/>
-        </gpio>
-        <gpio name="${tf_prefix}resend_robot_program">
-          <command_interface name="resend_robot_program_cmd"/>
-          <command_interface name="resend_robot_program_async_success"/>
-        </gpio>
-        <gpio name="${tf_prefix}hand_back_control">
-          <command_interface name="hand_back_control_cmd"/>
-          <command_interface name="hand_back_control_async_success"/>
-        </gpio>
-        <gpio name="${tf_prefix}zero_ftsensor">
-          <command_interface name="zero_ftsensor_cmd"/>
-          <command_interface name="zero_ftsensor_async_success"/>
-        </gpio>
-        <gpio name="${tf_prefix}system_interface">
-          <state_interface name="initialized"/>
-        </gpio>
-      </xacro:unless>
     </ros2_control>
   </xacro:macro>

File: install/hr_description/share/hr_description/urdf/hr.urdf.xacro (robot description, xacro)
@@ -3,9 +3,7 @@
     <!-- robot name parameter -->
     <xacro:arg name="name" default="hr"/>
-    <!-- import main macro -->
-    <xacro:include filename="$(find hr_description)/urdf/hr_macro.xacro"/>
     <!-- possible 'hr_type' values: ha006b, hh7, hh020, hs220_02, hx400, yl012 -->
     <!-- the default value should raise an error in case this was called without defining the type -->
-    <xacro:arg name="hr_type" default="hs220_02"/>
+    <xacro:arg name="hr_type" default="hx400"/>
     <!-- parameters -->
     <xacro:arg name="tf_prefix" default="" />
@@ -23,4 +21,5 @@
     <xacro:arg name="sim_ignition" default="false" />
     <xacro:arg name="simulation_controllers" default="" />
+    <xacro:arg name="use_conveyor_belt" default="false"/>
     <!-- initial position for simulations (Fake Hardware, Gazebo, Ignition) -->
     <xacro:arg name="initial_positions_file" default="$(find hr_description)/config/initial_positions.yaml"/>
@@ -29,24 +28,53 @@
     <!-- create link fixed to the "world" -->
     <link name="world" />
-    <!-- arm -->
-    <xacro:hr_robot
-        name="$(arg name)"
-        tf_prefix="$(arg tf_prefix)"
-        parent="world"
-        joint_limits_parameters_file="$(arg joint_limit_params)"
-        kinematics_parameters_file="$(arg kinematics_params)"
-        physical_parameters_file="$(arg physical_params)"
-        visual_parameters_file="$(arg visual_params)"
-        transmission_hw_interface="$(arg transmission_hw_interface)"
-        safety_limits="$(arg safety_limits)"
-        safety_pos_margin="$(arg safety_pos_margin)"
-        safety_k_position="$(arg safety_k_position)"
-        use_fake_hardware="$(arg use_fake_hardware)"
-        sim_gazebo="$(arg sim_gazebo)"
-        sim_ignition="$(arg sim_ignition)"
-        initial_positions="${xacro.load_yaml(initial_positions_file)}"
-        >
-        <origin xyz="0 0 0" rpy="0 0 0" />          <!-- position robot in the world -->
-    </xacro:hr_robot>
+    <!-- Conditional include based on hr_type -->
+    <xacro:if value="${'$(arg hr_type)' == 'hx400'}">
+        <!-- Include the HX400 parallel robot URDF -->
+        <xacro:include filename="$(find hr_description)/urdf/hr_macro_hx400.urdf"/>
+        <xacro:hr_parallel_robot
+            name="$(arg name)"
+            tf_prefix="$(arg tf_prefix)"
+            parent="world"
+            joint_limits_parameters_file="$(arg joint_limit_params)"
+            kinematics_parameters_file="$(arg kinematics_params)"
+            physical_parameters_file="$(arg physical_params)"
+            visual_parameters_file="$(arg visual_params)"
+            transmission_hw_interface="$(arg transmission_hw_interface)"
+            safety_limits="$(arg safety_limits)"
+            safety_pos_margin="$(arg safety_pos_margin)"
+            safety_k_position="$(arg safety_k_position)"
+            use_fake_hardware="$(arg use_fake_hardware)"
+            sim_gazebo="$(arg sim_gazebo)"
+            sim_ignition="$(arg sim_ignition)"
+            initial_positions="${xacro.load_yaml(initial_positions_file)}"
+            >
+            <origin xyz="0 0 0" rpy="0 0 0" />          <!-- position robot in the world -->
+        </xacro:hr_parallel_robot>
+    </xacro:if>
+    <xacro:unless value="${'$(arg hr_type)' == 'hx400'}">
+        <!-- import main macro for other robot types -->
+        <xacro:include filename="$(find hr_description)/urdf/hr_macro.xacro"/>
+        <!-- arm -->
+        <xacro:hr_robot
+            name="$(arg name)"
+            tf_prefix="$(arg tf_prefix)"
+            parent="world"
+            joint_limits_parameters_file="$(arg joint_limit_params)"
+            kinematics_parameters_file="$(arg kinematics_params)"
+            physical_parameters_file="$(arg physical_params)"
+            visual_parameters_file="$(arg visual_params)"
+            transmission_hw_interface="$(arg transmission_hw_interface)"
+            safety_limits="$(arg safety_limits)"
+            safety_pos_margin="$(arg safety_pos_margin)"
+            safety_k_position="$(arg safety_k_position)"
+            use_fake_hardware="$(arg use_fake_hardware)"
+            sim_gazebo="$(arg sim_gazebo)"
+            sim_ignition="$(arg sim_ignition)"
+            initial_positions="${xacro.load_yaml(initial_positions_file)}"
+            use_conveyor_belt="$(arg use_conveyor_belt)"
+            >
+            <origin xyz="0 0 0" rpy="0 0 0" />          <!-- position robot in the world -->
+        </xacro:hr_robot>
+    </xacro:unless>
     <xacro:if value="$(arg sim_gazebo)">
         <!-- Gazebo plugins -->

File: install/hr_description/share/hr_description/urdf/hr_macro.xacro (robot description, xacro)
@@ -21,4 +21,5 @@
     sim_ignition:=false
     initial_positions:=${dict(shoulder_pan_joint=0.0,shoulder_lift_joint=-1.57,elbow_joint=0.0,wrist_1_joint=-1.57,wrist_2_joint=0.0,wrist_3_joint=0.0)}
+    use_conveyor_belt:=false
     ">
     <!-- Load configuration data from the provided .yaml files -->
@@ -40,5 +41,51 @@
         sim_ignition="${sim_ignition}"
         tf_prefix="${tf_prefix}"
+        use_conveyor_belt="${use_conveyor_belt}"
         />
+    </xacro:if>
+    <xacro:if value="${use_conveyor_belt}">
+      <xacro:property name="mesh_scale" value="0.001" />
+      <link name="${tf_prefix}hs165_base_link">
+        <visual>
+          <origin xyz="0 0 0" rpy="0 0 0"/>
+          <geometry>
+            <mesh filename="package://hr_description/meshes/hs165/visual/frame_3600.STL" scale="${mesh_scale} ${mesh_scale} ${mesh_scale}"/>
+          </geometry>
+          <material name="frame_color">
+            <color rgba="0.5137 0.5137 0.5137 1"/>
+          </material>
+        </visual>
+        <collision>
+          <origin xyz="0 0 0" rpy="0 0 0"/>
+            <geometry>
+              <!-- 충돌 지오메트리를 간단한 형태로 변경 -->
+              <box size="3.6 0.8 0.1"/>  <!-- 실제 크기에 맞게 조정 필요 -->
+            </geometry>
+        </collision>
+        <xacro:cylinder_inertial radius="${base_inertia_radius}" length="${base_inertia_length}" mass="${base_mass}">
+          <origin xyz="0 0 0" rpy="0 0 0" />
+        </xacro:cylinder_inertial>
+      </link>
+      <link name="${tf_prefix}hs165_base">
+        <visual>
+          <origin xyz="0 0 0" rpy="0 0 0"/>
+          <geometry>
+            <mesh filename="package://hr_description/meshes/hs165/visual/base_3600.STL" scale="${mesh_scale} ${mesh_scale} ${mesh_scale}"/>
+          </geometry>
+          <material name="base_color">
+            <color rgba="0.1255 0.5020 0.0039 1"/>
+          </material>
+        </visual>
+        <collision>
+          <origin xyz="0 0 0" rpy="0 0 0"/>
+            <geometry>
+              <!-- 충돌 지오메트리를 간단한 형태로 변경 -->
+              <box size="0.5 0.5 0.2"/>  <!-- 실제 크기에 맞게 조정 필요 -->
+            </geometry>
+        </collision>
+        <xacro:cylinder_inertial radius="${base_inertia_radius}" length="${base_inertia_length}" mass="${base_mass}">
+          <origin xyz="0 0 0" rpy="0 0 0" />
+        </xacro:cylinder_inertial>
+      </link>
     </xacro:if>
     <!-- links -  main serial chain -->
@@ -172,10 +219,32 @@
       </xacro:cylinder_inertial>
     </link>
-    <!-- base_joint fixes base_link to the environment -->
-    <joint name="${tf_prefix}base_joint" type="fixed">
-      <xacro:insert_block name="origin" />
-      <parent link="${parent}" />
-      <child link="${tf_prefix}base_link" />
-    </joint>
+    <xacro:if value="${use_conveyor_belt}">
+      <joint name="world_to_hs165_base_link" type="fixed">
+        <parent link="world"/>
+        <child link="${tf_prefix}hs165_base_link"/>
+        <origin xyz="0 0 0" rpy="0 0 0"/>
+      </joint>
+      <joint name="${tf_prefix}conveyor_to_robot_base" type="prismatic">
+        <parent link="${tf_prefix}hs165_base_link"/>
+        <child link="${tf_prefix}hs165_base"/>
+        <origin xyz="0 0 0.555" rpy="0 0 0"/>
+        <axis xyz="0 1 0"/>
+        <limit lower="-1.8" upper="1.8" effort="1000" velocity="1"/>
+        <dynamics damping="1.0" friction="1.0"/>
+      </joint>
+      <joint name="${tf_prefix}base_joint" type="fixed">
+        <parent link="${tf_prefix}hs165_base"/>
+        <child link="${tf_prefix}base_link"/>
+        <origin xyz="0 0 0.1" rpy="0 0 0"/>
+      </joint>
+    </xacro:if>
+    <xacro:unless value="${use_conveyor_belt}">
+      <!-- base_joint fixes base_link to the environment -->
+      <joint name="${tf_prefix}base_joint" type="fixed">
+        <xacro:insert_block name="origin" />
+        <parent link="${parent}" />
+        <child link="${tf_prefix}base_link" />
+      </joint>
+    </xacro:unless>
     <!-- joints - main serial chain -->
     <joint name="${tf_prefix}base_link-base_link_inertia" type="fixed">
@@ -193,5 +262,5 @@
       <child link="${tf_prefix}shoulder_link" />
       <origin xyz="${shoulder_x} ${shoulder_y} ${shoulder_z}" rpy="${shoulder_roll} ${shoulder_pitch} ${shoulder_yaw}" />
-      <axis xyz="0 0 1" />
+      <axis xyz="${shoulder_axis_x} ${shoulder_axis_y} ${shoulder_axis_z}" />
       <limit lower="${shoulder_pan_lower_limit}" upper="${shoulder_pan_upper_limit}"
         effort="${shoulder_pan_effort_limit}" velocity="${shoulder_pan_velocity_limit}"/>
@@ -205,5 +274,5 @@
       <child link="${tf_prefix}upper_arm_link" />
       <origin xyz="${upper_arm_x} ${upper_arm_y} ${upper_arm_z}" rpy="${upper_arm_roll} ${upper_arm_pitch} ${upper_arm_yaw}" />
-      <axis xyz="0 0 1" />
+      <axis xyz="${upper_arm_axis_x} ${upper_arm_axis_y} ${upper_arm_axis_z}" />
       <limit lower="${shoulder_lift_lower_limit}" upper="${shoulder_lift_upper_limit}"
         effort="${shoulder_lift_effort_limit}" velocity="${shoulder_lift_velocity_limit}"/>
@@ -217,5 +286,5 @@
       <child link="${tf_prefix}forearm_link" />
       <origin xyz="${forearm_x} ${forearm_y} ${forearm_z}" rpy="${forearm_roll} ${forearm_pitch} ${forearm_yaw}" />
-      <axis xyz="0 0 1" />
+      <axis xyz="${forearm_axis_x} ${forearm_axis_y} ${forearm_axis_z}" />
       <limit lower="${elbow_joint_lower_limit}" upper="${elbow_joint_upper_limit}"
         effort="${elbow_joint_effort_limit}" velocity="${elbow_joint_velocity_limit}"/>
@@ -229,5 +298,5 @@
       <child link="${tf_prefix}wrist_1_link" />
       <origin xyz="${wrist_1_x} ${wrist_1_y} ${wrist_1_z}" rpy="${wrist_1_roll} ${wrist_1_pitch} ${wrist_1_yaw}" />
-      <axis xyz="0 0 1" />
+      <axis xyz="${wrist_1_axis_x} ${wrist_1_axis_y} ${wrist_1_axis_z}" />
       <limit lower="${wrist_1_lower_limit}" upper="${wrist_1_upper_limit}"
         effort="${wrist_1_effort_limit}" velocity="${wrist_1_velocity_limit}"/>
@@ -241,5 +310,5 @@
       <child link="${tf_prefix}wrist_2_link" />
       <origin xyz="${wrist_2_x} ${wrist_2_y} ${wrist_2_z}" rpy="${wrist_2_roll} ${wrist_2_pitch} ${wrist_2_yaw}" />
-      <axis xyz="0 0 1" />
+      <axis xyz="${wrist_2_axis_x} ${wrist_2_axis_y} ${wrist_2_axis_z}" />
       <limit lower="${wrist_2_lower_limit}" upper="${wrist_2_upper_limit}"
              effort="${wrist_2_effort_limit}" velocity="${wrist_2_velocity_limit}"/>
@@ -253,5 +322,5 @@
       <child link="${tf_prefix}wrist_3_link" />
       <origin xyz="${wrist_3_x} ${wrist_3_y} ${wrist_3_z}" rpy="${wrist_3_roll} ${wrist_3_pitch} ${wrist_3_yaw}" />
-      <axis xyz="0 0 1" />
+      <axis xyz="${wrist_3_axis_x} ${wrist_3_axis_y} ${wrist_3_axis_z}" />
       <limit lower="${wrist_3_lower_limit}" upper="${wrist_3_upper_limit}"
              effort="${wrist_3_effort_limit}" velocity="${wrist_3_velocity_limit}"/>
