Commit message: 0826 update

File: install/hr_description/share/hr_description/urdf/inc/hr_common.xacro (robot description, xacro)
@@ -88,5 +88,5 @@
     <xacro:property name="a3" value="${sec_dh_parameters['a3']}" scope="parent"/>
     <xacro:property name="d4" value="${sec_dh_parameters['d4']}" scope="parent"/>
-    <!-- <xacro:property name="d5" value="${sec_dh_parameters['d5']}" scope="parent"/> -->
+    <xacro:property name="d5" value="${sec_dh_parameters['d5']}" scope="parent"/>
     <xacro:property name="d6" value="${sec_dh_parameters['d6']}" scope="parent"/>
     <!-- kinematics -->
@@ -97,4 +97,7 @@
     <xacro:property name="shoulder_pitch" value="${sec_kinematics['shoulder']['pitch']}" scope="parent"/>
     <xacro:property name="shoulder_yaw" value="${sec_kinematics['shoulder']['yaw']}" scope="parent"/>
+    <xacro:property name="shoulder_axis_x" value="${sec_kinematics['shoulder']['axis_x']}" scope="parent"/>
+    <xacro:property name="shoulder_axis_y" value="${sec_kinematics['shoulder']['axis_y']}" scope="parent"/>
+    <xacro:property name="shoulder_axis_z" value="${sec_kinematics['shoulder']['axis_z']}" scope="parent"/>
     <xacro:property name="upper_arm_x" value="${sec_kinematics['upper_arm']['x']}" scope="parent"/>
     <xacro:property name="upper_arm_y" value="${sec_kinematics['upper_arm']['y']}" scope="parent"/>
@@ -103,4 +106,7 @@
     <xacro:property name="upper_arm_pitch" value="${sec_kinematics['upper_arm']['pitch']}" scope="parent"/>
     <xacro:property name="upper_arm_yaw" value="${sec_kinematics['upper_arm']['yaw']}" scope="parent"/>
+    <xacro:property name="upper_arm_axis_x" value="${sec_kinematics['upper_arm']['axis_x']}" scope="parent"/>
+    <xacro:property name="upper_arm_axis_y" value="${sec_kinematics['upper_arm']['axis_y']}" scope="parent"/>
+    <xacro:property name="upper_arm_axis_z" value="${sec_kinematics['upper_arm']['axis_z']}" scope="parent"/>
     <xacro:property name="forearm_x" value="${sec_kinematics['forearm']['x']}" scope="parent"/>
     <xacro:property name="forearm_y" value="${sec_kinematics['forearm']['y']}" scope="parent"/>
@@ -109,4 +115,7 @@
     <xacro:property name="forearm_pitch" value="${sec_kinematics['forearm']['pitch']}" scope="parent"/>
     <xacro:property name="forearm_yaw" value="${sec_kinematics['forearm']['yaw']}" scope="parent"/>
+    <xacro:property name="forearm_axis_x" value="${sec_kinematics['forearm']['axis_x']}" scope="parent"/>
+    <xacro:property name="forearm_axis_y" value="${sec_kinematics['forearm']['axis_y']}" scope="parent"/>
+    <xacro:property name="forearm_axis_z" value="${sec_kinematics['forearm']['axis_z']}" scope="parent"/>
     <xacro:property name="wrist_1_x" value="${sec_kinematics['wrist_1']['x']}" scope="parent"/>
     <xacro:property name="wrist_1_y" value="${sec_kinematics['wrist_1']['y']}" scope="parent"/>
@@ -115,4 +124,7 @@
     <xacro:property name="wrist_1_pitch" value="${sec_kinematics['wrist_1']['pitch']}" scope="parent"/>
     <xacro:property name="wrist_1_yaw" value="${sec_kinematics['wrist_1']['yaw']}" scope="parent"/>
+    <xacro:property name="wrist_1_axis_x" value="${sec_kinematics['wrist_1']['axis_x']}" scope="parent"/>
+    <xacro:property name="wrist_1_axis_y" value="${sec_kinematics['wrist_1']['axis_y']}" scope="parent"/>
+    <xacro:property name="wrist_1_axis_z" value="${sec_kinematics['wrist_1']['axis_z']}" scope="parent"/>
     <xacro:property name="wrist_2_x" value="${sec_kinematics['wrist_2']['x']}" scope="parent"/>
     <xacro:property name="wrist_2_y" value="${sec_kinematics['wrist_2']['y']}" scope="parent"/>
@@ -121,4 +133,7 @@
     <xacro:property name="wrist_2_pitch" value="${sec_kinematics['wrist_2']['pitch']}" scope="parent"/>
     <xacro:property name="wrist_2_yaw" value="${sec_kinematics['wrist_2']['yaw']}" scope="parent"/>
+    <xacro:property name="wrist_2_axis_x" value="${sec_kinematics['wrist_2']['axis_x']}" scope="parent"/>
+    <xacro:property name="wrist_2_axis_y" value="${sec_kinematics['wrist_2']['axis_y']}" scope="parent"/>
+    <xacro:property name="wrist_2_axis_z" value="${sec_kinematics['wrist_2']['axis_z']}" scope="parent"/>
     <xacro:property name="wrist_3_x" value="${sec_kinematics['wrist_3']['x']}" scope="parent"/>
     <xacro:property name="wrist_3_y" value="${sec_kinematics['wrist_3']['y']}" scope="parent"/>
@@ -127,4 +142,7 @@
     <xacro:property name="wrist_3_pitch" value="${sec_kinematics['wrist_3']['pitch']}" scope="parent"/>
     <xacro:property name="wrist_3_yaw" value="${sec_kinematics['wrist_3']['yaw']}" scope="parent"/>
+    <xacro:property name="wrist_3_axis_x" value="${sec_kinematics['wrist_3']['axis_x']}" scope="parent"/>
+    <xacro:property name="wrist_3_axis_y" value="${sec_kinematics['wrist_3']['axis_y']}" scope="parent"/>
+    <xacro:property name="wrist_3_axis_z" value="${sec_kinematics['wrist_3']['axis_z']}" scope="parent"/>
     <!-- OFFSETS -->
     <xacro:property name="shoulder_offset" value="${sec_offsets['shoulder_offset']}" scope="parent"/>

File: install/hr_moveit_config/share/hr_moveit_config/srdf/hr.srdf.xacro (robot description, xacro)
@@ -5,5 +5,7 @@
   <!-- parameters -->
   <xacro:arg name="prefix" default="" />
+  <!-- conveyor belt parameter -->
+  <xacro:arg name="use_conveyor_belt" default="false" />
   <xacro:include filename="$(find hr_moveit_config)/srdf/hr_macro.srdf.xacro"/>
-  <xacro:hr_srdf name="$(arg name)" prefix="$(arg prefix)"/>
+  <xacro:hr_srdf name="$(arg name)" prefix="$(arg prefix)" use_conveyor_belt="$(arg use_conveyor_belt)"/>
 </robot>

File: install/hr_moveit_config/share/hr_moveit_config/srdf/hr_macro.srdf.xacro (robot description, xacro)
@@ -5,5 +5,5 @@
     A URDF file must exist for this robot as well, where the joints and the links that are referenced are defined
 -->
-  <xacro:macro name="hr_srdf" params="name prefix">
+  <xacro:macro name="hr_srdf" params="name prefix use_conveyor_belt:=false">
     <!--GROUPS - Representation of a set of joints and links. This can be useful for specifying DOF to plan for, defining arms, end effectors, etc-->
     <!--LINKS - When a link is specified, the parent joint of that link (if it exists) is automatically included-->
@@ -13,5 +13,13 @@
     <group name="${prefix}${name}_manipulator">
       <chain base_link="${prefix}base_link" tip_link="${prefix}tool0" />
+      <xacro:if value="${use_conveyor_belt}">
+        <joint name="${prefix}conveyor_to_robot_base" />
+      </xacro:if>
     </group>
+    <xacro:if value="${use_conveyor_belt}">
+      <group name="${prefix}conveyor">
+        <joint name="${prefix}conveyor_to_robot_base" />
+      </group>
+    </xacro:if>
     <!--GROUP STATES - Purpose - Define a named state for a particular group, in terms of joint values. This is useful to define states like 'folded arms'-->
     <group_state name="${prefix}home" group="${prefix}${name}_manipulator">
@@ -22,4 +30,7 @@
       <joint name="${prefix}wrist_2_joint" value="0" />
       <joint name="${prefix}wrist_3_joint" value="0" />
+      <xacro:if value="${use_conveyor_belt}">
+        <joint name="${prefix}conveyor_to_robot_base" value="0" />
+      </xacro:if>
     </group_state>
     <group_state name="${prefix}up" group="${prefix}${name}_manipulator">
@@ -30,4 +41,7 @@
       <joint name="${prefix}wrist_2_joint" value="0" />
       <joint name="${prefix}wrist_3_joint" value="0" />
+      <xacro:if value="${use_conveyor_belt}">
+        <joint name="${prefix}conveyor_to_robot_base" value="0" />
+      </xacro:if>
     </group_state>
     <group_state name="${prefix}test_configuration" group="${prefix}${name}_manipulator">
@@ -38,5 +52,13 @@
       <joint name="${prefix}wrist_2_joint" value="-1.6" />
       <joint name="${prefix}wrist_3_joint" value="-0.11" />
+      <xacro:if value="${use_conveyor_belt}">
+        <joint name="${prefix}conveyor_to_robot_base" value="0" />
+      </xacro:if>
     </group_state>
+    <xacro:if value="${use_conveyor_belt}">
+      <group_state name="${prefix}conveyor_home" group="${prefix}conveyor">
+        <joint name="${prefix}conveyor_to_robot_base" value="0" />
+      </group_state>
+    </xacro:if>
     <!--END EFFECTOR - Purpose - Represent information about an end effector.-->
     <!--VIRTUAL JOINT - Purpose - this element defines a virtual joint between a robot link and an external frame of reference (considered fixed with respect to the robot)-->
@@ -53,4 +75,8 @@
     <disable_collisions link1="${prefix}wrist_1_link" link2="${prefix}wrist_3_link" reason="Never" />
     <disable_collisions link1="${prefix}wrist_2_link" link2="${prefix}wrist_3_link" reason="Adjacent" />
+    <xacro:if value="${use_conveyor_belt}">
+      <disable_collisions link1="${prefix}base_link" link2="${prefix}conveyor_belt" reason="Never" />
+      <disable_collisions link1="${prefix}shoulder_link" link2="${prefix}conveyor_belt" reason="Never" />
+    </xacro:if>
   </xacro:macro>
 </robot>
