Commit message: hx400 urdf update

File: hr_description/urdf/hr.urdf.xacro (robot description, xacro)
@@ -6,4 +6,6 @@
     <!-- the default value should raise an error in case this was called without defining the type -->
     <xacro:arg name="hr_type" default="hx400"/>
+     <!-- Convert hr_type argument to a property -->
+    <xacro:property name="hr_type" value="$(arg hr_type)" />
     <!-- parameters -->
     <xacro:arg name="tf_prefix" default="" />
@@ -22,4 +24,13 @@
     <xacro:arg name="simulation_controllers" default="" />
     <xacro:arg name="use_conveyor_belt" default="false"/>
+    <!-- <xacro:property name="hr_type_lower" value="${hr_type.lower()}"/>
+    <xacro:property name="use_hx_model" value="${'hx' in hr_type_lower}"/> -->
+    <xacro:property name="hr_type_lower" value="${hr_type.lower()}"/>
+    <xacro:if value="${'hx' in hr_type_lower}">
+        <xacro:property name="use_hx_model" value="true"/>
+    </xacro:if>
+    <xacro:unless value="${'hx' in hr_type_lower}">
+        <xacro:property name="use_hx_model" value="false"/>
+    </xacro:unless>
     <!-- initial position for simulations (Fake Hardware, Gazebo, Ignition) -->
     <xacro:arg name="initial_positions_file" default="$(find hr_description)/config/initial_positions.yaml"/>
@@ -28,53 +39,28 @@
     <!-- create link fixed to the "world" -->
     <link name="world" />
-    <!-- Conditional include based on hr_type -->
-    <xacro:if value="${'$(arg hr_type)' == 'hx400'}">
-        <!-- Include the HX400 parallel robot URDF -->
-        <xacro:include filename="$(find hr_description)/urdf/hr_macro_hx400.urdf"/>
-        <xacro:hr_parallel_robot
-            name="$(arg name)"
-            tf_prefix="$(arg tf_prefix)"
-            parent="world"
-            joint_limits_parameters_file="$(arg joint_limit_params)"
-            kinematics_parameters_file="$(arg kinematics_params)"
-            physical_parameters_file="$(arg physical_params)"
-            visual_parameters_file="$(arg visual_params)"
-            transmission_hw_interface="$(arg transmission_hw_interface)"
-            safety_limits="$(arg safety_limits)"
-            safety_pos_margin="$(arg safety_pos_margin)"
-            safety_k_position="$(arg safety_k_position)"
-            use_fake_hardware="$(arg use_fake_hardware)"
-            sim_gazebo="$(arg sim_gazebo)"
-            sim_ignition="$(arg sim_ignition)"
-            initial_positions="${xacro.load_yaml(initial_positions_file)}"
-            >
-            <origin xyz="0 0 0" rpy="0 0 0" />          <!-- position robot in the world -->
-        </xacro:hr_parallel_robot>
-    </xacro:if>
-    <xacro:unless value="${'$(arg hr_type)' == 'hx400'}">
-        <!-- import main macro for other robot types -->
-        <xacro:include filename="$(find hr_description)/urdf/hr_macro.xacro"/>
-        <!-- arm -->
-        <xacro:hr_robot
-            name="$(arg name)"
-            tf_prefix="$(arg tf_prefix)"
-            parent="world"
-            joint_limits_parameters_file="$(arg joint_limit_params)"
-            kinematics_parameters_file="$(arg kinematics_params)"
-            physical_parameters_file="$(arg physical_params)"
-            visual_parameters_file="$(arg visual_params)"
-            transmission_hw_interface="$(arg transmission_hw_interface)"
-            safety_limits="$(arg safety_limits)"
-            safety_pos_margin="$(arg safety_pos_margin)"
-            safety_k_position="$(arg safety_k_position)"
-            use_fake_hardware="$(arg use_fake_hardware)"
-            sim_gazebo="$(arg sim_gazebo)"
-            sim_ignition="$(arg sim_ignition)"
-            initial_positions="${xacro.load_yaml(initial_positions_file)}"
-            use_conveyor_belt="$(arg use_conveyor_belt)"
-            >
-            <origin xyz="0 0 0" rpy="0 0 0" />          <!-- position robot in the world -->
-        </xacro:hr_robot>
-    </xacro:unless>
+    <!-- import main macro for other robot types -->
+    <xacro:include filename="$(find hr_description)/urdf/hr_macro.xacro"/>
+    <!-- arm -->
+    <xacro:hr_robot
+        name="$(arg name)"
+        tf_prefix="$(arg tf_prefix)"
+        parent="world"
+        joint_limits_parameters_file="$(arg joint_limit_params)"
+        kinematics_parameters_file="$(arg kinematics_params)"
+        physical_parameters_file="$(arg physical_params)"
+        visual_parameters_file="$(arg visual_params)"
+        transmission_hw_interface="$(arg transmission_hw_interface)"
+        safety_limits="$(arg safety_limits)"
+        safety_pos_margin="$(arg safety_pos_margin)"
+        safety_k_position="$(arg safety_k_position)"
+        use_fake_hardware="$(arg use_fake_hardware)"
+        sim_gazebo="$(arg sim_gazebo)"
+        sim_ignition="$(arg sim_ignition)"
+        initial_positions="${xacro.load_yaml(initial_positions_file)}"
+        use_conveyor_belt="$(arg use_conveyor_belt)"
+        use_hx_model="${use_hx_model}"
+        >
+        <origin xyz="0 0 0" rpy="0 0 0" />          <!-- position robot in the world -->
+    </xacro:hr_robot>
     <xacro:if value="$(arg sim_gazebo)">
         <!-- Gazebo plugins -->

File: hr_description/urdf/hr_macro.xacro (robot description, xacro)
@@ -22,6 +22,6 @@
     initial_positions:=${dict(shoulder_pan_joint=0.0,shoulder_lift_joint=-1.57,elbow_joint=0.0,wrist_1_joint=-1.57,wrist_2_joint=0.0,wrist_3_joint=0.0)}
     use_conveyor_belt:=false
+    use_hx_model:=false
     ">
-    <!-- Load configuration data from the provided .yaml files -->
     <xacro:read_model_data
       joint_limits_parameters_file="${joint_limits_parameters_file}"
@@ -29,5 +29,6 @@
       physical_parameters_file="${physical_parameters_file}"
       visual_parameters_file="${visual_parameters_file}"
-      force_abs_paths="${sim_gazebo or sim_ignition}"/>
+      force_abs_paths="${sim_gazebo or sim_ignition}"
+      use_hx_model="${use_hx_model}"/>
     <xacro:if value="${generate_ros2_control_tag}">
       <!-- ros2 control include -->
@@ -127,5 +128,4 @@
     <link name="${tf_prefix}upper_arm_link">
       <visual>
-        <origin xyz="0 0 ${shoulder_offset}" rpy="${pi/2} 0 ${-pi/2}"/>
         <geometry>
           <xacro:get_mesh name="upper_arm" type="visual"/>
@@ -133,5 +133,4 @@
       </visual>
       <collision>
-        <origin xyz="0 0 ${shoulder_offset}" rpy="${pi/2} 0 ${-pi/2}"/>
         <geometry>
           <xacro:get_mesh name="upper_arm" type="collision"/>
@@ -144,5 +143,4 @@
     <link name="${tf_prefix}forearm_link">
       <visual>
-        <origin xyz="0 0 ${elbow_offset}" rpy="${pi/2} 0 ${-pi/2}"/>
         <geometry>
           <xacro:get_mesh name="forearm" type="visual"/>
@@ -150,5 +148,4 @@
       </visual>
       <collision>
-        <origin xyz="0 0 ${elbow_offset}" rpy="${pi/2} 0 ${-pi/2}"/>
         <geometry>
           <xacro:get_mesh name="forearm" type="collision"/>
@@ -163,5 +160,4 @@
       <visual>
         <xacro:get_origin name="wrist_1" type="visual" />
-      	<!-- <origin xyz="0 0 ${visual_params}" rpy="${pi/2} ${pi/2} 0"/> -->
         <geometry>
           <xacro:get_mesh name="wrist_1" type="visual"/>
@@ -170,5 +166,4 @@
       <collision>
         <xacro:get_origin name="wrist_1" type="collision" />
-        <!-- <origin xyz="0 0 ${visual_params}" rpy="${pi/2} ${pi/2} 0"/>  -->
         <geometry>
           <xacro:get_mesh name="wrist_1" type="collision"/>
@@ -183,5 +178,4 @@
       <visual>
         <xacro:get_origin name="wrist_2" type="visual" />
-        <!-- <origin xyz="0 0 ${visual_params}" rpy="${pi/2} 0 0"/> -->
         <geometry>
           <xacro:get_mesh name="wrist_2" type="visual"/>
@@ -190,5 +184,4 @@
       <collision>
         <xacro:get_origin name="wrist_2" type="collision" />
-        <!-- <origin xyz="0 0 ${visual_params}" rpy="${pi/2} 0 0"/> -->
         <geometry>
           <xacro:get_mesh name="wrist_2" type="collision"/>
@@ -203,5 +196,4 @@
       <visual>
         <xacro:get_origin name="wrist_3" type="visual" />
-        <!-- <origin xyz="0 0 ${visual_params}" rpy="0 ${pi/2} 0"/> -->
         <geometry>
           <xacro:get_mesh name="wrist_3" type="visual"/>
@@ -210,5 +202,4 @@
       <collision>
         <xacro:get_origin name="wrist_3" type="collision" />
-        <!-- <origin xyz="0 0 ${visual_params}" rpy="0 ${pi/2}0"/> -->
         <geometry>
           <xacro:get_mesh name="wrist_3" type="collision"/>
@@ -363,4 +354,98 @@
       <child link="${tf_prefix}tool0"/>
     </joint>
+    <xacro:if value="${use_hx_model}">
+      <!-- hx model parrel link add -->
+      <link name="${tf_prefix}hinge_link">
+        <visual>
+          <origin xyz="0 0 0" rpy="0 0 0"/>
+          <geometry>
+            <xacro:get_mesh name="hinge" type="visual"/>
+          </geometry>
+        </visual>
+        <collision>
+          <origin xyz="0 0 0" rpy="0 0 0"/>
+          <geometry>
+            <xacro:get_mesh name="hinge" type="collision"/>
+          </geometry>
+        </collision>
+      </link>
+      <link name="${tf_prefix}v_link">
+        <visual>
+          <origin xyz="0 0 0" rpy="0 0 0"/>
+          <geometry>
+            <xacro:get_mesh name="v_link" type="visual"/>
+          </geometry>
+        </visual>
+        <collision>
+          <origin xyz="0 0 0" rpy="0 0 0"/>
+          <geometry>
+            <xacro:get_mesh name="v_link" type="collision"/>
+          </geometry>
+        </collision>
+      </link>
+      <joint name="${tf_prefix}upper_arm_to_hinge_joint" type="continuous">
+        <parent link="${tf_prefix}upper_arm_link" />
+        <child link="${tf_prefix}hinge_link" />
+        <origin xyz="${hinge_x} ${hinge_y} ${hinge_z}" rpy="${hinge_roll} ${hinge_pitch} ${hinge_yaw}" />
+        <axis xyz="${hinge_axis_x} ${hinge_axis_y} ${hinge_axis_z}" />
+        <mimic joint="${tf_prefix}elbow_joint" multiplier="1" offset="0"/>
+      </joint>
+      <joint name="${tf_prefix}foream_arm_to_v_link_joint" type="continuous">
+        <parent link="${tf_prefix}forearm_link" />
+        <child link="${tf_prefix}v_link" />
+        <origin xyz="${v_link_x} ${v_link_y} ${v_link_z}" rpy="${v_link_roll} ${v_link_pitch} ${v_link_yaw}" />
+        <axis xyz="${v_link_axis_x} ${v_link_axis_y} ${v_link_axis_z}" />
+        <mimic joint="${tf_prefix}elbow_joint" multiplier="0" offset="0"/>
+      </joint>
+      <joint name="${tf_prefix}hinge_to_v_link" type="continuous">
+        <parent link="${tf_prefix}hinge_link" />
+        <child link="${tf_prefix}v_link" />
+        <origin xyz="${hinge_to_v_link_x} ${hinge_to_v_link_y} ${hinge_to_v_link_z}" rpy="${hinge_to_v_link_roll} ${hinge_to_v_link_pitch} ${hinge_to_v_link_yaw}" />
+        <axis xyz="${hinge_to_v_link_axis_x} ${hinge_to_v_link_axis_y} ${hinge_to_v_link_axis_z}" />
+        <mimic joint="${tf_prefix}elbow_joint" multiplier="-1" offset="0"/>
+      </joint>
+      <link name="${tf_prefix}p_tube_link">
+        <visual>
+          <origin xyz="0 0 0" rpy="0 0 0"/>
+          <geometry>
+            <xacro:get_mesh name="p_tube" type="visual"/>
+          </geometry>
+        </visual>
+        <collision>
+          <origin xyz="0 0 0" rpy="0 0 0"/>
+          <geometry>
+            <xacro:get_mesh name="p_tube" type="collision"/>
+          </geometry>
+        </collision>
+      </link>
+      <link name="${tf_prefix}p_shaft_link">
+        <visual>
+          <origin xyz="0 0 0" rpy="0 0 0"/>
+          <geometry>
+            <xacro:get_mesh name="p_shaft" type="visual"/>
+          </geometry>
+        </visual>
+        <collision>
+          <origin xyz="0 0 0" rpy="0 0 0"/>
+          <geometry>
+            <xacro:get_mesh name="p_shaft" type="collision"/>
+          </geometry>
+        </collision>
+      </link>
+      <joint name="${tf_prefix}p_tube_joint" type="continuous">
+        <parent link="${tf_prefix}upper_arm_link" />
+        <child link="${tf_prefix}p_tube_link" />
+        <origin xyz="${p_tube_x} ${p_tube_y} ${p_tube_z}" rpy="${p_tube_roll} ${p_tube_pitch} ${p_tube_yaw}" />
+        <axis xyz="${p_tube_axis_x} ${p_tube_axis_y} ${p_tube_axis_z}" />
+        <mimic joint="${tf_prefix}elbow_joint" multiplier="0.18" offset="0"/>
+      </joint>
+      <joint name="${tf_prefix}p_shaft_joint" type="continuous">
+        <parent link="${tf_prefix}shoulder_link" />
+        <child link="${tf_prefix}p_shaft_link" />
+        <origin xyz="${p_shaft_x} ${p_shaft_y} ${p_shaft_z}" rpy="${p_shaft_roll} ${p_shaft_pitch} ${p_shaft_yaw}" />
+        <axis xyz="${p_shaft_axis_x} ${p_shaft_axis_y} ${p_shaft_axis_z}" />
+        <mimic joint="${tf_prefix}elbow_joint" multiplier="1.18" offset="0"/>
+      </joint>
+    </xacro:if>
   </xacro:macro>
 </robot>

File: hr_description/urdf/inc/hr_common.xacro (robot description, xacro)
@@ -1,4 +1,5 @@
 <?xml version="1.0"?>
 <robot xmlns:xacro="http://wiki.ros.org/xacro">
+  <xacro:arg name="use_hx_model" default="false"/>
   <!--
     NOTE the macros defined in this file are NOT part of the public API of this
@@ -43,5 +44,5 @@
             rpy="${visual_origin_rpy[0]} ${visual_origin_rpy[1]} ${visual_origin_rpy[2]}"/>
   </xacro:macro>
-  <xacro:macro name="read_model_data" params="joint_limits_parameters_file kinematics_parameters_file physical_parameters_file visual_parameters_file force_abs_paths">
+  <xacro:macro name="read_model_data" params="joint_limits_parameters_file kinematics_parameters_file physical_parameters_file visual_parameters_file force_abs_paths use_hx_model">
     <xacro:property name="force_abs_paths" value="${force_abs_paths}" scope="parent"/>
     <!-- Read .yaml files from disk, load content into properties -->
@@ -145,4 +146,51 @@
     <xacro:property name="wrist_3_axis_y" value="${sec_kinematics['wrist_3']['axis_y']}" scope="parent"/>
     <xacro:property name="wrist_3_axis_z" value="${sec_kinematics['wrist_3']['axis_z']}" scope="parent"/>
+    <xacro:if value="${use_hx_model}">
+      <xacro:property name="hinge_x" value="${sec_kinematics['hinge']['x']}" scope="parent"/>
+      <xacro:property name="hinge_y" value="${sec_kinematics['hinge']['y']}" scope="parent"/>
+      <xacro:property name="hinge_z" value="${sec_kinematics['hinge']['z']}" scope="parent"/>
+      <xacro:property name="hinge_roll" value="${sec_kinematics['hinge']['roll']}" scope="parent"/>
+      <xacro:property name="hinge_pitch" value="${sec_kinematics['hinge']['pitch']}" scope="parent"/>
+      <xacro:property name="hinge_yaw" value="${sec_kinematics['hinge']['yaw']}" scope="parent"/>
+      <xacro:property name="hinge_axis_x" value="${sec_kinematics['hinge']['axis_x']}" scope="parent"/>
+      <xacro:property name="hinge_axis_y" value="${sec_kinematics['hinge']['axis_y']}" scope="parent"/>
+      <xacro:property name="hinge_axis_z" value="${sec_kinematics['hinge']['axis_z']}" scope="parent"/>
+      <xacro:property name="v_link_x" value="${sec_kinematics['v_link']['x']}" scope="parent"/>
+      <xacro:property name="v_link_y" value="${sec_kinematics['v_link']['y']}" scope="parent"/>
+      <xacro:property name="v_link_z" value="${sec_kinematics['v_link']['z']}" scope="parent"/>
+      <xacro:property name="v_link_roll" value="${sec_kinematics['v_link']['roll']}" scope="parent"/>
+      <xacro:property name="v_link_pitch" value="${sec_kinematics['v_link']['pitch']}" scope="parent"/>
+      <xacro:property name="v_link_yaw" value="${sec_kinematics['v_link']['yaw']}" scope="parent"/>
+      <xacro:property name="v_link_axis_x" value="${sec_kinematics['v_link']['axis_x']}" scope="parent"/>
+      <xacro:property name="v_link_axis_y" value="${sec_kinematics['v_link']['axis_y']}" scope="parent"/>
+      <xacro:property name="v_link_axis_z" value="${sec_kinematics['v_link']['axis_z']}" scope="parent"/>
+      <xacro:property name="hinge_to_v_link_x" value="${sec_kinematics['hinge_to_v_link']['x']}" scope="parent"/>
+      <xacro:property name="hinge_to_v_link_y" value="${sec_kinematics['hinge_to_v_link']['y']}" scope="parent"/>
+      <xacro:property name="hinge_to_v_link_z" value="${sec_kinematics['hinge_to_v_link']['z']}" scope="parent"/>
+      <xacro:property name="hinge_to_v_link_roll" value="${sec_kinematics['hinge_to_v_link']['roll']}" scope="parent"/>
+      <xacro:property name="hinge_to_v_link_pitch" value="${sec_kinematics['hinge_to_v_link']['pitch']}" scope="parent"/>
+      <xacro:property name="hinge_to_v_link_yaw" value="${sec_kinematics['hinge_to_v_link']['yaw']}" scope="parent"/>
+      <xacro:property name="hinge_to_v_link_axis_x" value="${sec_kinematics['hinge_to_v_link']['axis_x']}" scope="parent"/>
+      <xacro:property name="hinge_to_v_link_axis_y" value="${sec_kinematics['hinge_to_v_link']['axis_y']}" scope="parent"/>
+      <xacro:property name="hinge_to_v_link_axis_z" value="${sec_kinematics['hinge_to_v_link']['axis_z']}" scope="parent"/>
+      <xacro:property name="p_tube_x" value="${sec_kinematics['p_tube']['x']}" scope="parent"/>
+      <xacro:property name="p_tube_y" value="${sec_kinematics['p_tube']['y']}" scope="parent"/>
+      <xacro:property name="p_tube_z" value="${sec_kinematics['p_tube']['z']}" scope="parent"/>
+      <xacro:property name="p_tube_roll" value="${sec_kinematics['p_tube']['roll']}" scope="parent"/>
+      <xacro:property name="p_tube_pitch" value="${sec_kinematics['p_tube']['pitch']}" scope="parent"/>
+      <xacro:property name="p_tube_yaw" value="${sec_kinematics['p_tube']['yaw']}" scope="parent"/>
+      <xacro:property name="p_tube_axis_x" value="${sec_kinematics['p_tube']['axis_x']}" scope="parent"/>
+      <xacro:property name="p_tube_axis_y" value="${sec_kinematics['p_tube']['axis_y']}" scope="parent"/>
+      <xacro:property name="p_tube_axis_z" value="${sec_kinematics['p_tube']['axis_z']}" scope="parent"/>
+      <xacro:property name="p_shaft_x" value="${sec_kinematics['p_shaft']['x']}" scope="parent"/>
+      <xacro:property name="p_shaft_y" value="${sec_kinematics['p_shaft']['y']}" scope="parent"/>
+      <xacro:property name="p_shaft_z" value="${sec_kinematics['p_shaft']['z']}" scope="parent"/>
+      <xacro:property name="p_shaft_roll" value="${sec_kinematics['p_shaft']['roll']}" scope="parent"/>
+      <xacro:property name="p_shaft_pitch" value="${sec_kinematics['p_shaft']['pitch']}" scope="parent"/>
+      <xacro:property name="p_shaft_yaw" value="${sec_kinematics['p_shaft']['yaw']}" scope="parent"/>
+      <xacro:property name="p_shaft_axis_x" value="${sec_kinematics['p_shaft']['axis_x']}" scope="parent"/>
+      <xacro:property name="p_shaft_axis_y" value="${sec_kinematics['p_shaft']['axis_y']}" scope="parent"/>
+      <xacro:property name="p_shaft_axis_z" value="${sec_kinematics['p_shaft']['axis_z']}" scope="parent"/>
+    </xacro:if>
     <!-- OFFSETS -->
     <xacro:property name="shoulder_offset" value="${sec_offsets['shoulder_offset']}" scope="parent"/>

File: hr_moveit_config/srdf/hr_macro.srdf.xacro (robot description, xacro)
@@ -75,4 +75,25 @@
     <disable_collisions link1="${prefix}wrist_1_link" link2="${prefix}wrist_3_link" reason="Never" />
     <disable_collisions link1="${prefix}wrist_2_link" link2="${prefix}wrist_3_link" reason="Adjacent" />
+    <!-- hinge_link 관련 -->
+    <disable_collisions link1="${prefix}hinge_link" link2="${prefix}upper_arm_link" reason="Adjacent" />
+    <disable_collisions link1="${prefix}hinge_link" link2="${prefix}forearm_link" reason="Never" />
+    <disable_collisions link1="${prefix}hinge_link" link2="${prefix}shoulder_link" reason="Never" />
+    <!-- v_link 관련 -->
+    <disable_collisions link1="${prefix}v_link" link2="${prefix}forearm_link" reason="Adjacent" />
+    <disable_collisions link1="${prefix}v_link" link2="${prefix}upper_arm_link" reason="Never" />
+    <disable_collisions link1="${prefix}v_link" link2="${prefix}wrist_1_link" reason="Never" />
+    <disable_collisions link1="${prefix}v_link" link2="${prefix}v_link" reason="Never" />
+    <!-- hinge_link와 v_link 사이 -->
+    <disable_collisions link1="${prefix}hinge_link" link2="${prefix}v_link" reason="Adjacent" />
+    <!-- p_tube_link 관련 -->
+    <disable_collisions link1="${prefix}p_tube_link" link2="${prefix}upper_arm_link" reason="Adjacent" />
+    <disable_collisions link1="${prefix}p_tube_link" link2="${prefix}shoulder_link" reason="Never" />
+    <disable_collisions link1="${prefix}p_tube_link" link2="${prefix}forearm_link" reason="Never" />
+    <!-- p_shaft_link 관련 -->
+    <disable_collisions link1="${prefix}p_shaft_link" link2="${prefix}shoulder_link" reason="Adjacent" />
+    <disable_collisions link1="${prefix}p_shaft_link" link2="${prefix}upper_arm_link" reason="Never" />
+    <disable_collisions link1="${prefix}p_shaft_link" link2="${prefix}base_link_inertia" reason="Never" />
+    <!-- p_tube_link와 p_shaft_link 사이 -->
+    <disable_collisions link1="${prefix}p_tube_link" link2="${prefix}p_shaft_link" reason="Never" />
     <xacro:if value="${use_conveyor_belt}">
       <disable_collisions link1="${prefix}base_link" link2="${prefix}conveyor_belt" reason="Never" />
